File: max7325_dev.sch (KiCad schematic (older format))
At the start: 0 parts

Commit message: schematic: Draw first part of a scheme
Signed-off-by: Sam Protsenko <joe.skb7@gmail.com>
Parts:
- added C1: 0.1uF, Capacitors_SMD:C_1206, symbol C
- added D1: LED, LEDs:LED_D5.0mm, symbol LED
- added DNP-R2, DNP-R3, R4, R5: 0R, Resistors_SMD:R_1206, symbol R
- added J1: Conn_01x06, Pin_Headers:Pin_Header_Straight_1x06_Pitch2.54mm, symbol Conn_01x06
- added JP1: Jumper_NC_Dual, Pin_Headers:Pin_Header_Straight_1x03_Pitch2.54mm, symbol Jumper_NC_Dual
- added MK1, MK2, MK3, MK4: Mounting_Hole_PAD, Mounting_Holes:MountingHole_3.2mm_M3_Pad, symbol Mounting_Hole_PAD
- added R1: 10k, Resistors_SMD:R_1206, symbol R
- added SW1: SW_Push, Buttons_Switches_THT:SW_PUSH_6mm, symbol SW_Push
- added U1: MAX7325AEG+, Housings_SSOP:QSOP-24_3.9x8.7mm_Pitch0.635mm, symbol MAX7325AEG+
Connections:
- new net: DNP-R2.2, R4.1, U1.21 (AD0)
- new net: DNP-R3.2, R5.1, U1.3 (AD2)
- new net +3V3: C1.1, DNP-R2.1, DNP-R3.1, J1.1 (Pin_1), R1.1, U1.24 (V+)
- new net GND: C1.2, J1.6 (Pin_6), MK1.1, MK2.1, MK3.1, MK4.1, R4.2, R5.2, U1.12 (GND)
- new net INT: J1.4 (Pin_4), R1.2, U1.1 (~INT)
- new net RST: J1.5 (Pin_5), U1.2 (~RST)
- new net SCL: J1.2 (Pin_2), U1.22 (SCL)
- new net SDA: J1.3 (Pin_3), U1.23 (SDA)

Commit message: schematic: Finish the schematic
Signed-off-by: Sam Protsenko <joe.skb7@gmail.com>
Parts:
- added D0, D1, D10, D11, D12, D13, D14, D15, D2, D3, D4, D5, D6, D7, D9: LED, LEDs:LED_D5.0mm, symbol LED
- added JP1, JP2, JP3, JP4, JP5, JP6, JP7: Jumper_NC_Dual, Pin_Headers:Pin_Header_Straight_1x03_Pitch2.54mm, symbol Jumper_NC_Dual
- added R0, R1, R10, R11, R12, R13, R14, R15, R2, R3, R4, R5, R6, R7, R8, R9: 220R, Resistors_SMD:R_1206, symbol R
- added R16, R22, R23, R24, R25, R26, R27, R28, R29: 10k, Resistors_SMD:R_1206, symbol R
- added SW0, SW1, SW2, SW3, SW4, SW5, SW6: SW_Push, Buttons_Switches_THT:SW_PUSH_6mm, symbol SW_Push
- renumbered D1 to D8, JP1 to JP0, R1 to R17, DNP-R2 to R18, DNP-R3 to R19, R4 to R20, R5 to R21, SW1 to SW7
Connections:
- net +3V3: now also D8.2 (A), D0.2 (A), D1.2 (A), D10.2 (A), D11.2 (A), D12.2 (A), D13.2 (A), D14.2 (A), D15.2 (A), D2.2 (A), D3.2 (A), D4.2 (A), D5.2 (A), D6.2 (A), D7.2 (A), D9.2 (A), R16.1, R22.1, R23.1, R24.1, R25.1, R26.1, R27.1, R28.1, R29.1
- net GND: now also SW7.2, SW0.2, SW1.2, SW2.2, SW3.2, SW4.2, SW5.2, SW6.2
- net RST: now also R16.2
- net P6: now reaches U1.10 (P6)
- net P6: now also JP6.2
- net P7: now reaches U1.11 (P7)
- net P7: now also JP7.2
- net O8: now reaches U1.13 (O8)
- net O8: now also R8.1
- net O9: now reaches U1.14 (O9)
- net O9: now also R9.1
- net O10: now reaches U1.15 (O10)
- net O10: now also R10.1
- net O11: now reaches U1.16 (O11)
- net O11: now also R11.1
- net O12: now reaches U1.17 (O12)
- net O12: now also R12.1
- net O13: now reaches U1.18 (O13)
- net O13: now also R13.1
- net O14: now reaches U1.19 (O14)
- net O14: now also R14.1
- net O15: now reaches U1.20 (O15)
- net O15: now also R15.1
- net P0: now reaches U1.4 (P0)
- net P0: now also JP0.2
- net P1: now reaches U1.5 (P1)
- net P1: now also JP1.2
- net P2: now reaches U1.6 (P2)
- net P2: now also JP2.2
- net P3: now reaches U1.7 (P3)
- net P3: now also JP3.2
- net P4: now reaches U1.8 (P4)
- net P4: now also JP4.2
- net P5: now reaches U1.9 (P5)
- net P5: now also JP5.2
- net at D8.1 (K): now also R8.2
- net at JP0.1: now also R0.1
- net at JP0.3: now also R22.2, SW0.1
- net at SW7.1: now also JP7.3, R29.2
- new net: D9.1 (K), R9.2
- new net: D10.1 (K), R10.2
- new net: D11.1 (K), R11.2
- new net: D12.1 (K), R12.2
- new net: D13.1 (K), R13.2
- new net: D14.1 (K), R14.2
- new net: D15.1 (K), R15.2
- new net: D0.1 (K), R0.2
- new net: JP1.1, R1.1
- new net: JP1.3, R23.2, SW1.1
- new net: D1.1 (K), R1.2
- new net: JP2.1, R2.1
- new net: JP2.3, R24.2, SW2.1
- new net: D2.1 (K), R2.2
- new net: JP3.1, R3.1
- new net: JP3.3, R25.2, SW3.1
- new net: D3.1 (K), R3.2
- new net: JP4.1, R4.1
- new net: JP4.3, R26.2, SW4.1
- new net: D4.1 (K), R4.2
- new net: JP5.1, R5.1
- new net: JP5.3, R27.2, SW5.1
- new net: D5.1 (K), R5.2
- new net: JP6.1, R6.1
- new net: JP6.3, R28.2, SW6.1
- new net: D6.1 (K), R6.2
- new net: JP7.1, R7.1
- new net: D7.1 (K), R7.2
Other:
- note added: "I2C addresses:\n - 0x68: P0-P7\n - 0x58: O8-O15"
- note added: "R0P-R7P"
- moved on the sheet: C1, D8, J1, JP0, MK1, MK2, MK3, MK4, R17, R18, R19, R20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

Commit message: schematic: Finalaze schematic changes
Signed-off-by: Sam Protsenko <joe.skb7@gmail.com>
Parts:
- renumbered R22 to R100, R23 to R101, R24 to R102, R25 to R103, R26 to R104, R27 to R105, R28 to R106, R29 to R107
Other:
- note added: "R100-R107"
- note removed: "R0P-R7P"
Changed lines of the file:
@@
 Sheet 1 1
 Title "MAX7325 Demo Board"
-Date "2018-04-06"
+Date "2018-04-07"
 Rev "A"
 Comp "Dark Engineering Initiative"
@@
 $EndComp
 $Comp
-L R R22
+L R R100
 U 1 1 5AC928AE
 P 8300 1050
-F 0 "R22" V 8380 1050 50  0001 C CNN
+F 0 "R100" V 8380 1050 50  0001 C CNN
 F 1 "10k" V 8300 1050 50  0000 C CNN
 F 2 "Resistors_SMD:R_1206" V 8230 1050 50  0001 C CNN
@@
 $EndComp
 $Comp
-L R R23
+L R R101
 U 1 1 5AC935BC
 P 8400 1050
-F 0 "R23" V 8480 1050 50  0001 C CNN
+F 0 "R101" V 8480 1050 50  0001 C CNN
 F 1 "10k" V 8400 1050 50  0000 C CNN
 F 2 "Resistors_SMD:R_1206" V 8330 1050 50  0001 C CNN
@@
 $EndComp
 $Comp
-L R R24
+L R R102
 U 1 1 5AC936D0
 P 8500 1050
-F 0 "R24" V 8580 1050 50  0001 C CNN
+F 0 "R102" V 8580 1050 50  0001 C CNN
 F 1 "10k" V 8500 1050 50  0000 C CNN
 F 2 "Resistors_SMD:R_1206" V 8430 1050 50  0001 C CNN
@@
 $EndComp
 $Comp
-L R R25
+L R R103
 U 1 1 5AC937AF
 P 8600 1050
-F 0 "R25" V 8680 1050 50  0001 C CNN
+F 0 "R103" V 8680 1050 50  0001 C CNN
 F 1 "10k" V 8600 1050 50  0000 C CNN
 F 2 "Resistors_SMD:R_1206" V 8530 1050 50  0001 C CNN
@@
 $EndComp
 $Comp
-L R R26
+L R R104
 U 1 1 5AC9388E
 P 8700 1050
-F 0 "R26" V 8780 1050 50  0001 C CNN
+F 0 "R104" V 8780 1050 50  0001 C CNN
 F 1 "10k" V 8700 1050 50  0000 C CNN
 F 2 "Resistors_SMD:R_1206" V 8630 1050 50  0001 C CNN
@@
 $EndComp
 $Comp
-L R R27
+L R R105
 U 1 1 5AC9396D
 P 8800 1050
-F 0 "R27" V 8880 1050 50  0001 C CNN
+F 0 "R105" V 8880 1050 50  0001 C CNN
 F 1 "10k" V 8800 1050 50  0000 C CNN
 F 2 "Resistors_SMD:R_1206" V 8730 1050 50  0001 C CNN
@@
 $EndComp
 $Comp
-L R R28
+L R R106
 U 1 1 5AC93A4C
 P 8900 1050
-F 0 "R28" V 8980 1050 50  0001 C CNN
+F 0 "R106" V 8980 1050 50  0001 C CNN
 F 1 "10k" V 8900 1050 50  0000 C CNN
 F 2 "Resistors_SMD:R_1206" V 8830 1050 50  0001 C CNN
@@
 $EndComp
 $Comp
-L R R29
+L R R107
 U 1 1 5AC93B2B
 P 9000 1050
-F 0 "R29" V 9080 1050 50  0001 C CNN
+F 0 "R107" V 9080 1050 50  0001 C CNN
 F 1 "10k" V 9000 1050 50  0000 C CNN
 F 2 "Resistors_SMD:R_1206" V 8930 1050 50  0001 C CNN
@@
 	1    0    0    -1
 $EndComp
-Text Notes 8500 750  0    60   ~ 0
-R0P-R7P
+Text Notes 8400 750  0    60   ~ 0
+R100-R107
 Text Notes 3000 900  0    60   ~ 0
 I2C addresses:\n - 0x68: P0-P7\n - 0x58: O8-O15

Commit message: Migrate to KiCad 5.0
Signed-off-by: Sam Protsenko <joe.skb7@gmail.com>
Parts:
- C1: footprint Capacitors_SMD:C_1206 -> Capacitor_SMD:C_1206_3216Metric; symbol C -> Device:C
- D0, D1, D10, D11, D12, D13, D14, D15, D2, D3, D4, D5, D6, D7, D8, D9: footprint LEDs:LED_D5.0mm -> LED_THT:LED_D5.0mm; symbol LED -> Device:LED
- J1: footprint Pin_Headers:Pin_Header_Straight_1x06_Pitch2.54mm -> Connector_PinHeader_2.54mm:PinHeader_1x06_P2.54mm_Vertical; symbol Conn_01x06 -> Connector_Generic:Conn_01x06
- JP0, JP1, JP2, JP3, JP4, JP5, JP6, JP7: footprint Pin_Headers:Pin_Header_Straight_1x03_Pitch2.54mm -> Connector_PinHeader_2.54mm:PinHeader_1x03_P2.54mm_Vertical; symbol Jumper_NC_Dual -> Device:Jumper_NC_Dual
- MK1, MK2, MK3, MK4: footprint Mounting_Holes:MountingHole_3.2mm_M3_Pad -> MountingHole:MountingHole_3.2mm_M3_Pad; symbol Mounting_Hole_PAD -> Mechanical:MountingHole_Pad
- R0, R1, R10, R100, R101, R102, R103, R104, R105, R106, R107, R11, R12, R13, R14, R15, R16, R17, R18, R19, R2, R20, R21, R3, R4, R5, R6, R7, R8, R9: footprint Resistors_SMD:R_1206 -> Resistor_SMD:R_1206_3216Metric; symbol R -> Device:R
- SW0, SW1, SW2, SW3, SW4, SW5, SW6, SW7: footprint Buttons_Switches_THT:SW_PUSH_6mm -> Button_Switch_THT:SW_PUSH_6mm; symbol SW_Push -> Switch:SW_Push
- U1: footprint Housings_SSOP:QSOP-24_3.9x8.7mm_Pitch0.635mm -> Package_SO:QSOP-24_3.9x8.7mm_P0.635mm; symbol MAX7325AEG+ -> Interface_Expansion:MAX7325AEG+
Connections:
- wire segments 128 -> 168
